Commit message: updated to the current status of the chair

File: urdf/wheelchair_iaslab_sensors.xacro (robot description, xacro)
@@ -5,10 +5,14 @@
     xmlns:interface="http://playerstage.sourceforge.net/gazebo/xmlschema/#interface"
     name="wheelchair_iaslab_sensors">
-<xacro:include filename="wheelchair_iaslab.xacro" />
-<!-- Laser Hokuyo properties -->
-<xacro:property name="laser_length" value="0.04" />
-<xacro:property name="laser_radius" value="0.035" />
-<xacro:property name="laser_mass" value="0.160" />
-  <!-- Laser Hokuyo-->
+    <xacro:include filename="wheelchair_iaslab.xacro" />
+    <xacro:property name="xpos"    value ="0.346609" />
+    <xacro:property name="ypos"    value ="0.295568" />
+    <xacro:property name="zcamera" value ="0.58" />
+    <xacro:property name="zlaser"  value ="0.66" />
+    <!-- Laser Hokuyo properties -->
+    <xacro:property name="laser_length" value="0.04"  />
+    <xacro:property name="laser_radius" value="0.035" />
+    <xacro:property name="laser_mass"   value="0.160" />
+    <!-- Laser Hokuyo-->
     <link name="$(arg prefix)hokuyo_laser_link_left" >
         <visual>
@@ -17,5 +21,5 @@
             </geometry>
             <material name="red">
-                <color rgba="255 0 0 1"/>
+                <color rgba="1 0 0 1"/>
             </material>
         </visual>
@@ -31,12 +35,8 @@
     </link>
     <joint name="$(arg prefix)base_laser_joint_left" type="fixed">
-        <!--<parent link="$(arg prefix)base_link"/>
+        <axis xyz="0 1 0"/>
+        <parent link="$(arg prefix)base_footprint"/>
         <child link="$(arg prefix)hokuyo_laser_link_left"/>
-        <origin xyz="${pillow_length/2 + 0.105} 0.295 ${base_height/2 + pillow_height - 0.035}" rpy="0 0 0" /> -->
-        <axis xyz="0 1 0"/>
-<parent link="$(arg prefix)base_footprint"/>
-        <child link="$(arg prefix)hokuyo_laser_link_left"/>
-        <!-- <origin xyz="0.346609  0.295568  0.645" rpy="0 0 0" /> -->
-         <origin xyz="0.346609  0.0  0.645" rpy="0 0 0" />
+        <origin xyz="${xpos}  ${ypos}  ${zlaser}" rpy="0 0 0" />
         <axis xyz="0 1 0"/>
     </joint>
@@ -47,5 +47,5 @@
             </geometry>
             <material name="red">
-                <color rgba="255 0 0 1"/>
+                <color rgba="1 0 0 1"/>
             </material>
         </visual>
@@ -61,24 +61,42 @@
     </link>
     <joint name="$(arg prefix)base_laser_joint_right" type="fixed">
-       <!-- <parent link="$(arg prefix)base_link"/>
+        <parent link="$(arg prefix)base_footprint"/>
         <child link="$(arg prefix)hokuyo_laser_link_right"/>
-        <origin xyz="${pillow_length/2 + 0.11}  -0.295 ${base_height/2 + pillow_height - 0.02}" rpy="0 0 0" />
-        <axis xyz="0 1 0"/>-->
-<parent link="$(arg prefix)base_footprint"/>
-        <child link="$(arg prefix)hokuyo_laser_link_right"/>
-        <origin xyz="0.346609  -0.295568  0.66" rpy="0 0 0" />
-        <axis xyz="0 1 0"/>-->
+        <origin xyz="${xpos} -${ypos} ${zlaser}" rpy="0 0 0" />
+        <axis xyz="0 1 0"/>
     </joint>
-<!-- Real sense stereo camera-->
-<xacro:include filename="$(find realsense2_description)/urdf/_d435.urdf.xacro" />
-<xacro:sensor_d435 name="stereo_camera" parent="$(arg prefix)base_footprint" >
-<origin xyz=" 0.308867 0.24485 0.8" rpy="0 0 0" />
-    <!--<origin xyz="${pillow_length/2 +0.04}  0.277 ${base_height/2 + pillow_height + 0.12}" rpy="0 0 0" />-->
-  </xacro:sensor_d435>
-<!-- Real sense LIDAR camera-->
-<xacro:include filename="$(find realsense2_description)/urdf/_l515.urdf.xacro" />
-<xacro:sensor_l515 name="lidar_camera" parent="$(arg prefix)base_footprint" >
-<origin xyz="0.302795 -0.0503142 0.705" rpy="0 0 0" />
-    <!--<origin xyz="${pillow_length/2 +0.115}  0 ${base_height/2 + pillow_height + 0.025}" rpy="0 0 0" />-->
-  </xacro:sensor_l515>
+    <link name="$(arg prefix)imu_link" >
+        <visual>
+            <geometry>
+                <cylinder length="${laser_length}" radius="${laser_radius}"/>
+            </geometry>
+            <material name="red">
+                <color rgba="1 0 0 1"/>
+            </material>
+        </visual>
+        <collision>
+            <geometry>
+                <cylinder length="${laser_length}" radius="${laser_radius}"/>
+            </geometry>
+        </collision>
+        <inertial>
+            <mass value="${laser_mass}" />
+            <xacro:cylinder_inertia m="${laser_mass}" r="${laser_radius}" h="${laser_length}" />
+        </inertial>
+    </link>
+    <joint name="$(arg prefix)imu_link_j" type="fixed">
+	<parent link="$(arg prefix)base_footprint"/>
+        <child link="$(arg prefix)imu_link"/>
+         <origin xyz="0.0  0.0  0.05" rpy="0 0 0" />
+        <axis xyz="0 1 0"/>
+    </joint>
+    <!-- Real sense stereo camera-->
+    <xacro:arg name="use_nominal_extrinsics" default="false" />
+    <xacro:include filename="$(find realsense2_description)/urdf/_d435.urdf.xacro" />
+    <xacro:sensor_d435 name="camera_left" parent="$(arg prefix)base_footprint">
+        <origin xyz="${xpos} ${ypos} ${zcamera}" rpy="0 0 0" />
+    </xacro:sensor_d435>
+    <xacro:sensor_d435 name="camera_right" parent="$(arg prefix)base_footprint">
+        <origin xyz="${xpos} -${ypos} ${zcamera}" rpy="0 0 0"/>
+    </xacro:sensor_d435>
 </robot>

Commit message: 11/07/24

File: urdf/wheelchair_iaslab_sensors.xacro (robot description, xacro)
@@ -100,3 +100,6 @@
         <origin xyz="${xpos} -${ypos} ${zcamera}" rpy="0 0 0"/>
     </xacro:sensor_d435>
+    <xacro:sensor_d435 name="camera_top" parent="$(arg prefix)base_footprint">
+        <origin xyz="-0.3 0.0 1.47" rpy="0 0.147 0"/>
+    </xacro:sensor_d435>
 </robot>
