Commit message: 05/11/25

File: urdf/wheelchair_iaslab.xacro (robot description, xacro)
@@ -52,4 +52,10 @@
                  izz="${1/2*m*r*r}" />
     </xacro:macro>
+    <xacro:macro name="sphere_inertia" params="m r">
+    <inertia
+        ixx="${2.0/5.0 * m * r * r}" ixy="0.0" ixz="0.0"
+        iyy="${2.0/5.0 * m * r * r}" iyz="0.0"
+        izz="${2.0/5.0 * m * r * r}" />
+    </xacro:macro>
     <!-- Links and joints definitions -->
     <!-- Footprint and base -->
@@ -155,4 +161,12 @@
             </geometry>
             <origin xyz="0 0 0" rpy="${M_PI/2} 0 0" />
+            <surface>
+                <friction>
+                    <ode>
+                    <mu>1.0</mu>
+                    <mu2>1.0</mu2>
+                    </ode>
+                </friction>
+            </surface>
         </collision>
     </link>
@@ -160,5 +174,5 @@
         <parent link="$(arg prefix)base_link" />
         <child link="$(arg prefix)left_main_wheel_link" />
-        <origin xyz="0.23  ${base_width/2 + main_wheel_length/2} -${base_height/2}" rpy="0 0 0" />
+        <origin xyz="0.23  ${base_width/2 + main_wheel_length/2 + 0.01} -${base_height/2}" rpy="0 0 0" />
         <axis xyz="0 1 0" />
         <joint_properties damping="0.0" friction="0.0" />
@@ -184,4 +198,12 @@
             </geometry>
             <origin xyz="0 0 0" rpy="${M_PI/2} 0 0" />
+            <surface>
+                <friction>
+                    <ode>
+                    <mu>1.0</mu>
+                    <mu2>1.0</mu2>
+                    </ode>
+                </friction>
+            </surface>
         </collision>
     </link>
@@ -189,9 +211,9 @@
         <parent link="$(arg prefix)base_link" />
         <child link="$(arg prefix)right_main_wheel_link" />
-        <origin xyz="0.23  -${base_width/2 + main_wheel_length/2} -${base_height/2}" rpy="0 0 0" />
+        <origin xyz="0.23  -${base_width/2 + main_wheel_length/2 + 0.01} -${base_height/2}" rpy="0 0 0" />
         <axis xyz="0 1 0" />
         <joint_properties damping="0.0" friction="0.0" />
     </joint>
-    <!-- Rear wheels -->
+    <!-- Rear wheels
     <link name="$(arg prefix)left_small_wheel_link">
         <inertial>
@@ -251,5 +273,182 @@
         <axis xyz="0 1 0" />
         <joint_properties damping="0.0" friction="0.0" />
-    </joint>
+    </joint> -->
     <!--The 0.07cm is the difference between the radius of the two wheels-->
+    <!-- Rear caster wheel
+    <link name="$(arg prefix)right_rear_caster_link">
+        <inertial>
+            <mass value="0.05"/>
+            <origin xyz="0 0 0"/>
+            <xacro:sphere_inertia m="0.05" r="0.03"/>
+        </inertial>
+        <visual>
+            <geometry>
+            <sphere radius="0.03"/>
+            </geometry>
+            <material name="black">
+            <color rgba="0 0 0 0.4"/>
+            </material>
+        </visual>
+        <collision>
+            <geometry>
+            <sphere radius="0.03"/>
+            </geometry>
+        </collision>
+    </link>
+    <joint name="$(arg prefix)right_rear_caster_joint" type="continuous">
+        <parent link="$(arg prefix)base_link"/>
+        <child link="$(arg prefix)right_rear_caster_link"/>
+        <origin xyz="-${base_length/2} -${base_width/2 + small_wheel_length/2} -${base_height/2 + 0.13}" rpy="0 0 0"/>
+        <axis xyz="0 0 1"/>
+        <joint_properties damping="0.5" friction="0.0" />
+    </joint>
+    <link name="$(arg prefix)left_rear_caster_link">
+        <inertial>
+            <mass value="0.05"/>
+            <origin xyz="0 0 0"/>
+            <xacro:sphere_inertia m="0.05" r="0.03"/>
+        </inertial>
+        <visual>
+            <geometry>
+            <sphere radius="0.03"/>
+            </geometry>
+            <material name="black">
+            <color rgba="0 0 0 0.4"/>
+            </material>
+        </visual>
+        <collision>
+            <geometry>
+            <sphere radius="0.03"/>
+            </geometry>
+        </collision>
+    </link>
+    <joint name="$(arg prefix)left_rear_caster_joint" type="continuous">
+        <parent link="$(arg prefix)base_link"/>
+        <child link="$(arg prefix)left_rear_caster_link"/>
+        <origin xyz="-${base_length/2} ${base_width/2 + small_wheel_length/2} -${base_height/2 + 0.13}" rpy="0 0 0"/>
+        <axis xyz="0 0 1"/>
+        <joint_properties damping="0.5" friction="0.0" />
+    </joint> -->
+    <!-- Swivel link (the caster fork) -->
+    <link name="$(arg prefix)left_caster_swivel_link">
+    <inertial>
+        <mass value="0.05"/>
+        <origin xyz="0 0 0"/>
+        <xacro:sphere_inertia m="0.05" r="0.02"/>
+    </inertial>
+    <visual>
+        <geometry>
+            <sphere radius="0.02"/>
+        </geometry>
+        <material name="grey">
+            <color rgba="0.5 0.5 0.5 1.0"/>
+        </material>
+    </visual>
+        <collision>
+            <geometry>
+                <sphere radius="0.02"/>
+            </geometry>
+        </collision>
+    </link>
+    <joint name="$(arg prefix)left_rear_caster_joint" type="continuous">
+        <parent link="$(arg prefix)base_link"/>
+        <child link="$(arg prefix)left_caster_swivel_link"/>
+        <origin xyz="-${base_length/2} ${base_width/2 + small_wheel_length/2 +0.07} 0" rpy="0 0 0"/>
+        <axis xyz="0 0 1"/>
+      <!-- <joint_properties damping="0.5" friction="0.0" /> -->
+    </joint>
+    <!-- Wheel link -->
+    <link name="$(arg prefix)left_rear_caster_link">
+        <inertial>
+            <mass value="0.05"/>
+            <origin xyz="0 0 0"/>
+            <!-- <xacro:cylinder_inertia m="0.05" r="${small_wheel_radius}" h="${small_wheel_length}"/> -->
+            <xacro:sphere_inertia m="0.5" r="${small_wheel_radius/2}"/>
+        </inertial>
+        <visual>
+            <geometry>
+                <!-- <cylinder length="${small_wheel_length}" radius="${small_wheel_radius}"/> -->
+                <sphere radius="${small_wheel_radius/2}"/>
+            </geometry>
+            <material name="grey">
+                <color rgba="0.5 0.5 0.5 1.0"/>
+            </material>
+            <origin xyz="0 0 0" rpy="${M_PI/2} 0 0"/>
+        </visual>
+        <collision>
+            <geometry>
+                <!-- <cylinder length="${small_wheel_length}" radius="${small_wheel_radius}"/> -->
+                <sphere radius="${small_wheel_radius/2}"/>
+            </geometry>
+            <origin xyz="0 0 0" rpy="${M_PI/2} 0 0"/>
+        </collision>
+    </link>
+    <!-- Wheel spin joint -->
+    <joint name="$(arg prefix)left_caster_spin_joint" type="continuous">
+        <parent link="$(arg prefix)left_caster_swivel_link"/>
+        <child link="$(arg prefix)left_rear_caster_link"/>
+        <origin xyz="0 0 -${small_wheel_radius/2 + 0.27}" rpy="0 0 0"/>
+        <axis xyz="0 1 0"/>
+    </joint>
+    <!-- Swivel link (the caster fork) -->
+    <link name="$(arg prefix)right_caster_swivel_link">
+        <inertial>
+            <mass value="0.05"/>
+            <origin xyz="0 0 0"/>
+            <xacro:sphere_inertia m="0.05" r="0.02"/>
+        </inertial>
+        <visual>
+            <geometry>
+                <sphere radius="0.02"/>
+            </geometry>
+            <material name="grey">
+                <color rgba="0.5 0.5 0.5 1.0"/>
+            </material>
+        </visual>
+        <collision>
+            <geometry>
+                <sphere radius="0.02"/>
+            </geometry>
+        </collision>
+    </link>
+    <joint name="$(arg prefix)right_rear_caster_joint" type="continuous">
+        <parent link="$(arg prefix)base_link"/>
+        <child link="$(arg prefix)right_caster_swivel_link"/>
+        <origin xyz="-${base_length/2} -${base_width/2 + small_wheel_length/2 +0.07} 0" rpy="0 0 0"/>
+        <axis xyz="0 0 1"/>
+      <!-- <joint_properties damping="0.5" friction="0.0" /> -->
+    </joint>
+    <!-- Wheel link -->
+    <link name="$(arg prefix)right_rear_caster_link">
+        <inertial>
+            <mass value="0.05"/>
+            <origin xyz="0 0 0"/>
+            <!-- <xacro:cylinder_inertia m="0.05" r="${small_wheel_radius}" h="${small_wheel_length}"/> -->
+            <xacro:sphere_inertia m="0.5" r="${small_wheel_radius/2}"/>
+        </inertial>
+        <visual>
+            <geometry>
+                <!-- <cylinder length="${small_wheel_length}" radius="${small_wheel_radius}"/> -->
+                <sphere radius="${small_wheel_radius/2}"/>
+            </geometry>
+            <material name="grey">
+                <color rgba="0.5 0.5 0.5 1.0"/>
+            </material>
+            <origin xyz="0 0 0" rpy="${M_PI/2} 0 0"/>
+        </visual>
+        <collision>
+            <geometry>
+                <!-- <cylinder length="${small_wheel_length}" radius="${small_wheel_radius}"/> -->
+                <sphere radius="${small_wheel_radius/2}"/>
+            </geometry>
+            <origin xyz="0 0 0" rpy="${M_PI/2} 0 0"/>
+        </collision>
+    </link>
+    <!-- Wheel spin joint -->
+    <joint name="$(arg prefix)rigth_caster_spin_joint" type="continuous">
+        <parent link="$(arg prefix)right_caster_swivel_link"/>
+        <child link="$(arg prefix)right_rear_caster_link"/>
+        <origin xyz="0 0 -${small_wheel_radius/2 + 0.27}" rpy="0 0 0"/>
+        <axis xyz="0 1 0"/>
+    </joint>
 </robot>

File: urdf/wheelchair_iaslab_sensors.xacro (robot description, xacro)
@@ -6,8 +6,9 @@
     name="wheelchair_iaslab_sensors">
     <xacro:include filename="wheelchair_iaslab.xacro" />
-    <xacro:property name="xpos"    value ="0.346609" />
-    <xacro:property name="ypos"    value ="0.295568" />
+    <xacro:property name="xpos"    value ="0.45" />
+    <xacro:property name="ypos"    value ="0.30" />
     <xacro:property name="zcamera" value ="0.58" />
-    <xacro:property name="zlaser"  value ="0.66" />
+    <xacro:property name="zlaser"  value ="0.58" />
+    <xacro:property name="rotylaser"  value ="1.57" />
     <!-- Laser Hokuyo properties -->
     <xacro:property name="laser_length" value="0.04"  />
@@ -38,5 +39,5 @@
         <parent link="$(arg prefix)base_footprint"/>
         <child link="$(arg prefix)hokuyo_laser_link_left"/>
-        <origin xyz="${xpos}  ${ypos}  ${zlaser}" rpy="0 0 0" />
+        <origin xyz="${xpos}  ${ypos}  ${zlaser}" rpy="0 0 ${rotylaser}" />
         <axis xyz="0 1 0"/>
     </joint>
@@ -63,5 +64,5 @@
         <parent link="$(arg prefix)base_footprint"/>
         <child link="$(arg prefix)hokuyo_laser_link_right"/>
-        <origin xyz="${xpos} -${ypos} ${zlaser}" rpy="0 0 0" />
+        <origin xyz="${xpos} -${ypos} ${zlaser}" rpy="0 0 -${rotylaser}" />
         <axis xyz="0 1 0"/>
     </joint>
